Commit message: Bee 1 robot modeli ve sensor eklentileri duzeltildi

File: Arac_Ws/install/bee1_description/share/bee1_description/urdf/bee1.xacro (robot description, xacro)
@@ -1,87 +1 @@
-<?xml version="1.0"?>
-<robot name="bee1" xmlns:xacro="http://www.ros.org/wiki/xacro">
-  <xacro:property name="wheel_radius" value="0.265" />
-  <xacro:property name="wheel_width" value="0.15" />
-  <xacro:property name="wheelbase" value="1.860" />
-  <xacro:property name="front_track" value="0.886" />
-  <xacro:property name="rear_track" value="0.850" />
-  <link name="base_footprint"/>
-  <joint name="base_joint" type="fixed">
-    <parent link="base_footprint"/>
-    <child link="base_link"/>
-    <origin xyz="0 0 ${wheel_radius}" rpy="0 0 0"/>
-  </joint>
-  <link name="base_link">
-    <visual>
-      <origin xyz="${wheelbase / 2.0} 0 0.1" rpy="0 0 0"/>
-      <geometry><box size="2.74 1.06 0.2"/></geometry>
-      <material name="white"><color rgba="1 1 1 1"/></material>
-    </visual>
-    <visual>
-      <origin xyz="1.0 0 0.7" rpy="0 0 0"/>
-      <geometry><box size="1.0 1.0 1.2"/></geometry>
-    </visual>
-    <visual>
-      <origin xyz="1.9 0 0.3" rpy="0 0.2 0"/>
-      <geometry><box size="0.8 1.0 0.6"/></geometry>
-    </visual>
-    <visual>
-      <origin xyz="0.1 0 0.7" rpy="0 0 0"/>
-      <geometry><box size="0.8 1.0 1.2"/></geometry>
-    </visual>
-    <collision>
-      <origin xyz="${wheelbase / 2.0} 0 0.5" rpy="0 0 0"/>
-      <geometry><box size="2.74 1.06 1.0"/></geometry>
-    </collision>
-    <inertial>
-      <origin xyz="0.7 0 0.3" rpy="0 0 0"/>
-      <mass value="760.0"/>
-      <inertia ixx="100.0" ixy="0.0" ixz="0.0" iyy="100.0" iyz="0.0" izz="100.0"/>
-    </inertial>
-  </link>
-  <xacro:macro name="wheel" params="prefix x y">
-    <link name="${prefix}_wheel">
-      <visual>
-        <origin xyz="0 0 0" rpy="${pi/2} 0 0"/>
-        <geometry><cylinder length="${wheel_width}" radius="${wheel_radius}"/></geometry>
-        <material name="black"><color rgba="0 0 0 1"/></material>
-      </visual>
-      <collision>
-        <origin xyz="0 0 0" rpy="${pi/2} 0 0"/>
-        <geometry><cylinder length="${wheel_width}" radius="${wheel_radius}"/></geometry>
-      </collision>
-      <inertial>
-        <mass value="15.0"/>
-        <inertia ixx="0.1" ixy="0" ixz="0" iyy="0.1" iyz="0" izz="0.1"/>
-      </inertial>
-    </link>
-    <joint name="${prefix}_wheel_joint" type="continuous">
-      <parent link="base_link"/>
-      <child link="${prefix}_wheel"/>
-      <origin xyz="${x} ${y} 0" rpy="0 0 0"/>
-      <axis xyz="0 1 0"/>
-    </joint>
-  </xacro:macro>
-  <xacro:wheel prefix="rear_right" x="0" y="-${rear_track/2}"/>
-  <xacro:wheel prefix="rear_left"  x="0" y="${rear_track/2}"/>
-  <xacro:wheel prefix="front_right" x="${wheelbase}" y="-${front_track/2}"/>
-  <xacro:wheel prefix="front_left"  x="${wheelbase}" y="${front_track/2}"/>
-  <gazebo>
-    <plugin name='diff_drive' filename='libgazebo_ros_diff_drive.so'>
-      <ros>
-        <namespace>/</namespace>
-      </ros>
-      <left_joint>rear_left_wheel_joint</left_joint>
-      <right_joint>rear_right_wheel_joint</right_joint>
-      <wheel_separation>${rear_track}</wheel_separation>
-      <wheel_diameter>${wheel_radius * 2}</wheel_diameter>
-      <max_wheel_torque>200</max_wheel_torque>
-      <max_wheel_acceleration>10.0</max_wheel_acceleration>
-      <odometry_frame>odom</odometry_frame>
-      <robot_base_frame>base_footprint</robot_base_frame>
-      <publish_odom>true</publish_odom>
-      <publish_odom_tf>true</publish_odom_tf>
-      <publish_wheel_tf>true</publish_wheel_tf>
-    </plugin>
-  </gazebo>
-</robot>
+/home/zeynep/Desktop/Arac_Ws/src/bee1_description/urdf/bee1.xacro

Commit message: Map modelleri ve world dosyası eklendi

File: Arac_Ws/install/bee1_description/share/bee1_description/urdf/bee1.xacro (robot description, xacro)
@@ -1 +1,140 @@
-/home/zeynep/Desktop/Arac_Ws/src/bee1_description/urdf/bee1.xacro
+<?xml version="1.0"?>
+<robot name="bee1" xmlns:xacro="http://www.ros.org/wiki/xacro">
+  <xacro:property name="wheel_radius" value="0.265" />
+  <xacro:property name="wheel_width" value="0.15" />
+  <xacro:property name="wheelbase" value="1.860" />
+  <xacro:property name="front_track" value="0.886" />
+  <xacro:property name="rear_track" value="0.850" />
+  <link name="base_footprint"/>
+  <joint name="base_joint" type="fixed">
+    <parent link="base_footprint"/>
+    <child link="base_link"/>
+    <origin xyz="0 0 ${wheel_radius}" rpy="0 0 0"/>
+  </joint>
+  <link name="base_link">
+    <visual>
+      <origin xyz="${wheelbase / 2.0} 0 0.1" rpy="0 0 0"/>
+      <geometry><box size="2.74 1.06 0.2"/></geometry>
+      <material name="white"><color rgba="1 1 1 1"/></material>
+    </visual>
+    <visual>
+      <origin xyz="1.0 0 0.7" rpy="0 0 0"/>
+      <geometry><box size="1.0 1.0 1.2"/></geometry>
+    </visual>
+    <visual>
+      <origin xyz="1.9 0 0.3" rpy="0 0.2 0"/>
+      <geometry><box size="0.8 1.0 0.6"/></geometry>
+    </visual>
+    <visual>
+      <origin xyz="0.1 0 0.7" rpy="0 0 0"/>
+      <geometry><box size="0.8 1.0 1.2"/></geometry>
+    </visual>
+    <collision>
+      <origin xyz="${wheelbase / 2.0} 0 0.5" rpy="0 0 0"/>
+      <geometry><box size="2.74 1.06 1.0"/></geometry>
+    </collision>
+    <inertial>
+      <origin xyz="0.7 0 0.3" rpy="0 0 0"/>
+      <mass value="760.0"/>
+      <inertia ixx="100.0" ixy="0.0" ixz="0.0" iyy="100.0" iyz="0.0" izz="100.0"/>
+    </inertial>
+  </link>
+  <xacro:macro name="wheel" params="prefix x y">
+    <link name="${prefix}_wheel">
+      <visual>
+        <origin xyz="0 0 0" rpy="${pi/2} 0 0"/>
+        <geometry><cylinder length="${wheel_width}" radius="${wheel_radius}"/></geometry>
+        <material name="black"><color rgba="0 0 0 1"/></material>
+      </visual>
+      <collision>
+        <origin xyz="0 0 0" rpy="${pi/2} 0 0"/>
+        <geometry><cylinder length="${wheel_width}" radius="${wheel_radius}"/></geometry>
+      </collision>
+      <inertial>
+        <mass value="15.0"/>
+        <inertia ixx="0.1" ixy="0" ixz="0" iyy="0.1" iyz="0" izz="0.1"/>
+      </inertial>
+    </link>
+    <joint name="${prefix}_wheel_joint" type="continuous">
+      <parent link="base_link"/>
+      <child link="${prefix}_wheel"/>
+      <origin xyz="${x} ${y} 0" rpy="0 0 0"/>
+      <axis xyz="0 1 0"/>
+    </joint>
+  </xacro:macro>
+  <xacro:wheel prefix="rear_right" x="0" y="-${rear_track/2}"/>
+  <xacro:wheel prefix="rear_left"  x="0" y="${rear_track/2}"/>
+  <xacro:wheel prefix="front_right" x="${wheelbase}" y="-${front_track/2}"/>
+  <xacro:wheel prefix="front_left"  x="${wheelbase}" y="${front_track/2}"/>
+  <!-- SENSÖRLER[cite: 1] -->
+  <link name="lidar_link">
+    <visual><geometry><cylinder radius="0.05" length="0.07"/></geometry></visual>
+  </link>
+  <joint name="lidar_joint" type="fixed">
+    <parent link="base_link"/>
+    <child link="lidar_link"/>
+    <origin xyz="${wheelbase - 0.177} 0 0.620" rpy="0 0 0"/>
+  </joint>
+  <link name="camera_left_link">
+    <visual><geometry><box size="0.03 0.03 0.03"/></geometry></visual>
+  </link>
+  <joint name="camera_left_joint" type="fixed">
+    <parent link="base_link"/>
+    <child link="camera_left_link"/>
+    <origin xyz="${wheelbase + 0.205} 0.060 0.685" rpy="0 0 0"/>
+  </joint>
+  <link name="imu_gps_link">
+    <visual><geometry><box size="0.05 0.05 0.02"/></geometry></visual>
+  </link>
+  <joint name="imu_gps_joint" type="fixed">
+    <parent link="base_link"/>
+    <child link="imu_gps_link"/>
+    <origin xyz="${wheelbase + 1.440} 0 1.390" rpy="0 0 0"/>
+  </joint>
+  <!-- GAZEBO EKLENTİLERİ -->
+  <gazebo>
+    <plugin name='diff_drive' filename='libgazebo_ros_diff_drive.so'>
+      <ros><namespace>/</namespace></ros>
+      <left_joint>rear_left_wheel_joint</left_joint>
+      <right_joint>rear_right_wheel_joint</right_joint>
+      <wheel_separation>${rear_track}</wheel_separation>
+      <wheel_diameter>${wheel_radius * 2}</wheel_diameter>
+      <max_wheel_torque>200</max_wheel_torque>
+      <max_wheel_acceleration>10.0</max_wheel_acceleration>
+      <odometry_frame>odom</odometry_frame>
+      <robot_base_frame>base_footprint</robot_base_frame>
+      <publish_odom>true</publish_odom>
+      <publish_odom_tf>true</publish_odom_tf>
+      <publish_wheel_tf>true</publish_wheel_tf>
+    </plugin>
+  </gazebo>
+  <gazebo reference="lidar_link">
+    <sensor type="ray" name="velodyne_vlp16">
+      <pose>0 0 0 0 0 0</pose>
+      <visualize>true</visualize>
+      <update_rate>10</update_rate>
+      <ray>
+        <scan>
+          <horizontal><samples>440</samples><resolution>1</resolution><min_angle>-3.14</min_angle><max_angle>3.14</max_angle></horizontal>
+          <vertical><samples>16</samples><resolution>1</resolution><min_angle>-0.26</min_angle><max_angle>0.26</max_angle></vertical>
+        </scan>
+        <range><min>0.3</min><max>100.0</max><resolution>0.001</resolution></range>
+      </ray>
+      <!-- DOSYA ADI ÇOK ÖNEMLİ: libgazebo_ros_velodyne_laser.so -->
+      <plugin name="lidar_controller" filename="libgazebo_ros_velodyne_laser.so">
+        <ros>
+          <remapping>~/out:=/velodyne_points</remapping>
+        </ros>
+        <frame_name>lidar_link</frame_name>
+      </plugin>
+    </sensor>
+  </gazebo>
+  <gazebo reference="imu_gps_link">
+    <plugin name="imu_plugin" filename="libgazebo_ros_imu_sensor.so">
+      <ros>
+        <namespace>/</namespace>
+        <remapping>~/out:=imu/data</remapping>
+      </ros>
+    </plugin>
+  </gazebo>
+</robot>

Commit message: Lidar range 0.8 yapildi, IMU ve kamera sensorleri eklendi

File: Arac_Ws/install/bee1_description/share/bee1_description/urdf/bee1.xacro (robot description, xacro)
@@ -74,5 +74,5 @@
       <cylinder radius="0.05" length="0.07"/>
     </geometry>
-    <material name="black"/>
+    <material name="black"><color rgba="0 0 0 1"/></material>
   </visual>
 </link>
@@ -89,5 +89,5 @@
       <box size="0.03 0.17 0.03"/>
     </geometry>
-    <material name="grey"/>
+    <material name="grey"><color rgba="0.5 0.5 0.5 1"/></material>
   </visual>
 </link>
@@ -103,5 +103,5 @@
       <box size="0.03 0.17 0.03"/>
     </geometry>
-    <material name="grey"/>
+    <material name="grey"><color rgba="0.5 0.5 0.5 1"/></material>
   </visual>
 </link>
@@ -117,5 +117,5 @@
       <box size="0.05 0.05 0.02"/>
     </geometry>
-    <material name="red"/>
+    <material name="red"><color rgba="1 0 0 1"/></material>
   </visual>
 </link>
@@ -125,4 +125,16 @@
   <origin xyz="-1.440 0.0 1.390" rpy="0 0 0"/>
 </joint>
+<!-- 4. IMU Link (Yeni Eklendi) -->
+  <link name="imu_link">
+    <visual>
+      <geometry><box size="0.05 0.05 0.02"/></geometry>
+      <material name="orange"><color rgba="1.0 0.5 0.0 1"/></material>
+    </visual>
+  </link>
+  <joint name="imu_joint" type="fixed">
+    <parent link="base_link"/>
+    <child link="imu_link"/>
+    <origin xyz="0 0 0" rpy="0 0 0"/> <!-- Genelde merkeze yakın yerleştirilir -->
+  </joint>
   <!-- GAZEBO EKLENTİLERİ -->
   <gazebo>
@@ -158,5 +170,5 @@
       </scan>
       <range>
-        <min>0.3</min>
+        <min>0.8</min>
         <max>100.0</max>
       </range>
@@ -170,4 +182,17 @@
     </plugin>
   </sensor>
+</gazebo>
+<gazebo reference="imu_link">
+    <sensor name="imu_sensor" type="imu">
+      <always_on>true</always_on>
+      <update_rate>100</update_rate>
+      <visualize>true</visualize>
+      <plugin name="imu_controller" filename="libgazebo_ros_imu_sensor.so">
+        <ros>
+          <remapping>~/out:=imu</remapping>
+        </ros>
+        <initial_orientation_as_reference>false</initial_orientation_as_reference>
+      </plugin>
+    </sensor>
 </gazebo>
 <gazebo reference="gps_link">
